File: AP_KACA.sch (EAGLE design)
At the start: 50 parts, among them IC1 REG710XX-3.3, J1 FTDI_DEVICE, M1 WIRELESS-NRF24L01, Q1 BSS123, Q2 BSS123, Q3 BSS123, Q4 BSS123, U3 GY-521MPU6050, Y1 8MHz

Commit message: Updated schematic
Parts:
- removed C10: 0.22uF, we-rcl:CAPACITOR-1206
- removed C11, C12: 2.2uF, we-rcl:CAPACITOR-1206
- removed IC1: REG710XX-3.3, we-power:REG710XX-3.3
- added C13, C14: 1uF, we-rcl:CAPACITOR-0603
- added VOLTAGEREG: SPX3819M5_3_3, SparkFun-IC-Power:V_REG_SPX3819-SOT23-5
Connections:
- removed net N$10: C10.2, IC1.C+
- removed net N$11: C10.1, IC1.C-
- new net N$14: C13.2, VOLTAGEREG.OUT
- net 3.3V: no longer C11.2, IC1.VOUT
- net 3.7V: now also C14.2, VOLTAGEREG.EN, VOLTAGEREG.IN; no longer C12.1, IC1.EN, IC1.VIN
- net DGND: now also C13.1, C14.1, U1.GND@5, VOLTAGEREG.GND; no longer C11.1, C12.2, IC1.GND
Changed lines of the file:
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@@
 <layers>
 <layer number="1" name="Top" color="4" fill="1" visible="no" active="no"/>
+<layer number="2" name="Route2" color="1" fill="3" visible="no" active="no"/>
+<layer number="3" name="Route3" color="4" fill="3" visible="no" active="no"/>
+<layer number="4" name="Route4" color="1" fill="4" visible="no" active="no"/>
+<layer number="5" name="Route5" color="4" fill="4" visible="no" active="no"/>
+<layer number="6" name="Route6" color="1" fill="8" visible="no" active="no"/>
+<layer number="7" name="Route7" color="4" fill="8" visible="no" active="no"/>
+<layer number="8" name="Route8" color="1" fill="2" visible="no" active="no"/>
+<layer number="9" name="Route9" color="4" fill="2" visible="no" active="no"/>
+<layer number="10" name="Route10" color="1" fill="7" visible="no" active="no"/>
+<layer number="11" name="Route11" color="4" fill="7" visible="no" active="no"/>
+<layer number="12" name="Route12" color="1" fill="5" visible="no" active="no"/>
+<layer number="13" name="Route13" color="4" fill="5" visible="no" active="no"/>
+<layer number="14" name="Route14" color="1" fill="6" visible="no" active="no"/>
+<layer number="15" name="Route15" color="4" fill="6" visible="no" active="no"/>
 <layer number="16" name="Bottom" color="1" fill="1" visible="no" active="no"/>
 <layer number="17" name="Pads" color="2" fill="1" visible="no" active="no"/>
@@
 <part name="Q1" library="transistor-small-signal" deviceset="BSS123" device=""/>
 <part name="D1" library="diode" deviceset="ES2D" device=""/>
-<part name="IC1" library="we-power" deviceset="REG710XX" device="-3.3"/>
 <part name="U$2" library="JST_CONNECTOR_FEMALE. through hole" deviceset="JST_CONNECTOR_FEMALE" device=""/>
 <part name="J1" library="quad" deviceset="FTDI_DEVICE" device=""/>
@@
 <part name="LED1" library="eagle-ltspice" deviceset="LED_E" device="SML0603"/>
 <part name="R2" library="SparkFun-Resistors" deviceset="10.5KOHM1/10W1%(0603)" device="" value="510"/>
-<part name="C10" library="we-rcl" deviceset="CAPACITOR" device="-1206" value="0.22uF"/>
-<part name="C11" library="we-rcl" deviceset="CAPACITOR" device="-1206" value="2.2uF"/>
-<part name="C12" library="we-rcl" deviceset="CAPACITOR" device="-1206" value="2.2uF"/>
 <part name="R3" library="SparkFun-Resistors" deviceset="10.5KOHM1/10W1%(0603)" device="" value="36k"/>
 <part name="Q2" library="transistor-small-signal" deviceset="BSS123" device=""/>
@@
 <part name="U$7" library="splitter" deviceset="SPLITTER" device=""/>
 <part name="U$8" library="splitter" deviceset="SPLITTER" device=""/>
+<part name="VOLTAGEREG" library="SparkFun-IC-Power" deviceset="V_REG_SPX3819" device="-SOT23-5" value="SPX3819M5_3_3"/>
+<part name="C13" library="we-rcl" deviceset="CAPACITOR" device="-0603" value="1uF"/>
+<part name="C14" library="we-rcl" deviceset="CAPACITOR" device="-0603" value="1uF"/>
 </parts>
 <sheets>
@@
 <instance part="Q1" gate="G$1" x="-45.72" y="83.82"/>
 <instance part="D1" gate="G$1" x="-45.72" y="99.06" rot="R90"/>
-<instance part="IC1" gate="IC" x="248.92" y="35.56"/>
 <instance part="U$2" gate="G$1" x="251.46" y="63.5" rot="R180"/>
 <instance part="J1" gate="G$1" x="48.26" y="101.6" rot="R180"/>
@@
 <instance part="LED1" gate="G$1" x="246.38" y="81.28" rot="R270"/>
 <instance part="R2" gate="G$1" x="233.68" y="81.28"/>
-<instance part="C10" gate="C" x="271.78" y="35.56" rot="R90"/>
-<instance part="C11" gate="C" x="269.24" y="48.26" rot="R180"/>
-<instance part="C12" gate="C" x="228.6" y="48.26" rot="R180"/>
 <instance part="R3" gate="G$1" x="-40.64" y="73.66" rot="R90"/>
 <instance part="Q2" gate="G$1" x="-91.44" y="83.82"/>
@@
 <instance part="U$7" gate="G$1" x="236.22" y="106.68"/>
 <instance part="U$8" gate="G$1" x="236.22" y="121.92"/>
+<instance part="VOLTAGEREG" gate="G$1" x="167.64" y="111.76"/>
+<instance part="C13" gate="C" x="182.88" y="114.3" rot="R90"/>
+<instance part="C14" gate="C" x="152.4" y="114.3" rot="R90"/>
 </instances>
 <busses>
@@
 </segment>
 <segment>
-<pinref part="IC1" gate="IC" pin="VOUT"/>
-<wire x1="261.62" y1="43.18" x2="264.16" y2="43.18" width="0.1524" layer="91"/>
-<label x="274.32" y="43.18" size="1.778" layer="95" xref="yes"/>
-<wire x1="264.16" y1="43.18" x2="274.32" y2="43.18" width="0.1524" layer="91"/>
-<wire x1="264.16" y1="43.18" x2="264.16" y2="48.26" width="0.1524" layer="91"/>
-<junction x="264.16" y="43.18"/>
-<pinref part="C11" gate="C" pin="2"/>
-<wire x1="266.7" y1="48.26" x2="264.16" y2="48.26" width="0.1524" layer="91"/>
-</segment>
-<segment>
 <pinref part="R1" gate="G$1" pin="2"/>
 <wire x1="60.96" y1="129.54" x2="66.04" y2="129.54" width="0.1524" layer="91"/>
@@
 <pinref part="U1" gate="U$1" pin="GND@3"/>
 <pinref part="U1" gate="U$1" pin="GND@PAD"/>
-<wire x1="30.48" y1="27.94" x2="30.48" y2="22.86" width="0.1524" layer="91"/>
+<wire x1="30.48" y1="27.94" x2="30.48" y2="25.4" width="0.1524" layer="91"/>
+<wire x1="30.48" y1="25.4" x2="30.48" y2="22.86" width="0.1524" layer="91"/>
 <wire x1="30.48" y1="22.86" x2="27.94" y2="22.86" width="0.1524" layer="91"/>
 <junction x="30.48" y="22.86"/>
 <label x="27.94" y="22.86" size="1.778" layer="95" rot="R180" xref="yes"/>
+<pinref part="U1" gate="U$1" pin="GND@5"/>
+<junction x="30.48" y="25.4"/>
 </segment>
 <segment>
@@
 </segment>
 <segment>
-<pinref part="IC1" gate="IC" pin="GND"/>
-<wire x1="248.92" y1="27.94" x2="248.92" y2="25.4" width="0.1524" layer="91"/>
-<wire x1="248.92" y1="25.4" x2="246.38" y2="25.4" width="0.1524" layer="91"/>
-<label x="246.38" y="25.4" size="1.778" layer="95" rot="R180" xref="yes"/>
-</segment>
-<segment>
-<pinref part="C11" gate="C" pin="1"/>
-<wire x1="271.78" y1="48.26" x2="274.32" y2="48.26" width="0.1524" layer="91"/>
-<label x="274.32" y="48.26" size="1.778" layer="95" xref="yes"/>
-</segment>
-<segment>
-<pinref part="C12" gate="C" pin="2"/>
-<wire x1="226.06" y1="48.26" x2="223.52" y2="48.26" width="0.1524" layer="91"/>
-<label x="223.52" y="48.26" size="1.778" layer="95" rot="R180" xref="yes"/>
-</segment>
-<segment>
 <pinref part="R7" gate="G$1" pin="2"/>
 <wire x1="60.96" y1="10.16" x2="66.04" y2="10.16" width="0.1524" layer="91"/>
@@
 <wire x1="241.3" y1="121.92" x2="248.92" y2="121.92" width="0.1524" layer="91"/>
 <label x="248.92" y="121.92" size="1.778" layer="95" xref="yes"/>
+</segment>
+<segment>
+<pinref part="C14" gate="C" pin="1"/>
+<pinref part="VOLTAGEREG" gate="G$1" pin="GND"/>
+<wire x1="152.4" y1="111.76" x2="157.48" y2="111.76" width="0.1524" layer="91"/>
+<label x="139.7" y="111.76" size="1.778" layer="95" rot="R180" xref="yes"/>
+<wire x1="152.4" y1="111.76" x2="139.7" y2="111.76" width="0.1524" layer="91"/>
+<junction x="152.4" y="111.76"/>
+</segment>
+<segment>
+<pinref part="C13" gate="C" pin="1"/>
+<wire x1="182.88" y1="111.76" x2="182.88" y2="109.22" width="0.1524" layer="91"/>
+<label x="182.88" y="109.22" size="1.778" layer="95" xref="yes"/>
 </segment>
 </net>
@@
 <pinref part="U$1" gate="G$1" pin="+"/>
 <wire x1="-33.02" y1="99.06" x2="-27.94" y2="99.06" width="0.1524" layer="91"/>
-</segment>
-<segment>
-<pinref part="IC1" gate="IC" pin="VIN"/>
-<wire x1="236.22" y1="43.18" x2="233.68" y2="43.18" width="0.1524" layer="91"/>
-<label x="223.52" y="43.18" size="1.778" layer="95" rot="R180" xref="yes"/>
-<wire x1="233.68" y1="43.18" x2="223.52" y2="43.18" width="0.1524" layer="91"/>
-<wire x1="233.68" y1="43.18" x2="233.68" y2="33.02" width="0.1524" layer="91"/>
-<junction x="233.68" y="43.18"/>
-<pinref part="IC1" gate="IC" pin="EN"/>
-<wire x1="233.68" y1="33.02" x2="236.22" y2="33.02" width="0.1524" layer="91"/>
-<wire x1="233.68" y1="43.18" x2="233.68" y2="48.26" width="0.1524" layer="91"/>
-<wire x1="233.68" y1="48.26" x2="231.14" y2="48.26" width="0.1524" layer="91"/>
-<pinref part="C12" gate="C" pin="1"/>
 </segment>
 <segment>
@@
 <label x="279.4" y="96.52" size="1.778" layer="95" xref="yes"/>
 </segment>
+<segment>
+<pinref part="VOLTAGEREG" gate="G$1" pin="EN"/>
+<wire x1="157.48" y1="106.68" x2="152.4" y2="106.68" width="0.1524" layer="91"/>
+<label x="152.4" y="106.68" size="1.778" layer="95" rot="R180" xref="yes"/>
+</segment>
+<segment>
+<pinref part="C14" gate="C" pin="2"/>
+<pinref part="VOLTAGEREG" gate="G$1" pin="IN"/>
+<wire x1="152.4" y1="116.84" x2="157.48" y2="116.84" width="0.1524" layer="91"/>
+<wire x1="152.4" y1="116.84" x2="152.4" y2="121.92" width="0.1524" layer="91"/>
+<junction x="152.4" y="116.84"/>
+<label x="152.4" y="121.92" size="1.778" layer="95" rot="R180" xref="yes"/>
+</segment>
 </net>
 <net name="MGND" class="0">
@@
 <wire x1="241.3" y1="81.28" x2="238.76" y2="81.28" width="0.1524" layer="91"/>
 <pinref part="R2" gate="G$1" pin="2"/>
-</segment>
-</net>
-<net name="N$11" class="0">
-<segment>
-<pinref part="IC1" gate="IC" pin="C-"/>
-<wire x1="261.62" y1="33.02" x2="261.62" y2="30.48" width="0.1524" layer="91"/>
-<wire x1="261.62" y1="30.48" x2="271.78" y2="30.48" width="0.1524" layer="91"/>
-<wire x1="271.78" y1="30.48" x2="271.78" y2="33.02" width="0.1524" layer="91"/>
-<pinref part="C10" gate="C" pin="1"/>
-</segment>
-</net>
-<net name="N$10" class="0">
-<segment>
-<pinref part="IC1" gate="IC" pin="C+"/>
-<wire x1="261.62" y1="38.1" x2="261.62" y2="40.64" width="0.1524" layer="91"/>
-<pinref part="C10" gate="C" pin="2"/>
-<wire x1="261.62" y1="40.64" x2="271.78" y2="40.64" width="0.1524" layer="91"/>
-<wire x1="271.78" y1="40.64" x2="271.78" y2="38.1" width="0.1524" layer="91"/>
 </segment>
 </net>
@@
 </segment>
 </net>
+<net name="N$14" class="0">
+<segment>
+<pinref part="VOLTAGEREG" gate="G$1" pin="OUT"/>
+<pinref part="C13" gate="C" pin="2"/>
+<wire x1="175.26" y1="116.84" x2="182.88" y2="116.84" width="0.1524" layer="91"/>
+</segment>
+</net>

Commit message: lol
Connections:
- removed net N$12: C4.2, U1.AVCC
- removed net N$14: C13.2, VOLTAGEREG.OUT
- net 3.3V: now also C13.2, C4.2, U1.AVCC, VOLTAGEREG.OUT
Changed lines of the file:
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@@
 <label x="66.04" y="129.54" size="1.778" layer="95" xref="yes"/>
+</segment>
+<segment>
+<pinref part="C4" gate="C" pin="2"/>
+<wire x1="12.7" y1="86.36" x2="22.86" y2="86.36" width="0.1524" layer="91"/>
+<pinref part="U1" gate="U$1" pin="AVCC"/>
+<wire x1="22.86" y1="86.36" x2="22.86" y2="76.2" width="0.1524" layer="91"/>
+<wire x1="22.86" y1="76.2" x2="30.48" y2="76.2" width="0.1524" layer="91"/>
+<wire x1="22.86" y1="86.36" x2="22.86" y2="91.44" width="0.1524" layer="91"/>
+<junction x="22.86" y="86.36"/>
+<label x="22.86" y="91.44" size="1.778" layer="95" rot="R180" xref="yes"/>
+</segment>
+<segment>
+<pinref part="VOLTAGEREG" gate="G$1" pin="OUT"/>
+<pinref part="C13" gate="C" pin="2"/>
+<wire x1="175.26" y1="116.84" x2="182.88" y2="116.84" width="0.1524" layer="91"/>
+<wire x1="182.88" y1="116.84" x2="182.88" y2="121.92" width="0.1524" layer="91"/>
+<junction x="182.88" y="116.84"/>
+<label x="182.88" y="121.92" size="1.778" layer="95" xref="yes"/>
 </segment>
 </net>
@@
 </segment>
 </net>
-<net name="N$12" class="0">
-<segment>
-<pinref part="C4" gate="C" pin="2"/>
-<wire x1="12.7" y1="86.36" x2="22.86" y2="86.36" width="0.1524" layer="91"/>
-<pinref part="U1" gate="U$1" pin="AVCC"/>
-<wire x1="22.86" y1="86.36" x2="22.86" y2="76.2" width="0.1524" layer="91"/>
-<wire x1="22.86" y1="76.2" x2="30.48" y2="76.2" width="0.1524" layer="91"/>
-</segment>
-</net>
 <net name="N$9" class="0">
 <segment>
@@
 </segment>
 </net>
-<net name="N$14" class="0">
-<segment>
-<pinref part="VOLTAGEREG" gate="G$1" pin="OUT"/>
-<pinref part="C13" gate="C" pin="2"/>
-<wire x1="175.26" y1="116.84" x2="182.88" y2="116.84" width="0.1524" layer="91"/>
-</segment>
-</net>
