File: AP_KACA.sch (EAGLE design)
At the start: 49 parts, among them J1 FTDI_DEVICE, M1 WIRELESS-NRF24L01, Q1 BSS123, Q2 BSS123, Q3 BSS123, Q4 BSS123, U3 GY-521MPU6050, Y1 8MHz

Commit message: Update SCH
Parts:
- removed C1, C2: 36pF, we-rcl:CAPACITOR-0603
- removed VOLTAGEREG: SPX3819M5_3_3, SparkFun-IC-Power:V_REG_SPX3819-SOT23-5
- added C10: 1uF, we-rcl:CAPACITOR-0603
- added C11: 10uF, we-rcl:CAPACITOR-0603
- added C12: 60pF, OPS_Project_6_LIB:RCL_C-USC1206
- added IC1: MCP1252-33X50, microchip-MCP125x-xxx:MCP1252-33X50
- C13: value 1uF -> 60pF; device we-rcl:CAPACITOR-0603 -> OPS_Project_6_LIB:RCL_C-USC1206
- C14: value 1uF -> 10uF
- R10, R11, R3, R4, R5, R6: value 36k -> 10k
- U1: value (none) -> ATMEGA328P_TQFP; device SparkFun-DigitalIC:ATMEGA328P_MLFMLF32 -> quad:ATMEGA328P_TQFP
Connections:
- removed net CTS: J1.CTS
- new net N$11: C10.2, IC1.C-
- new net N$12: C10.1, IC1.C+
- net 3.3V: now also C14.2, IC1.VOUT; no longer C13.2, VOLTAGEREG.OUT
- net 3.7V: now also C11.2, IC1.SELECT, IC1.SHDN, IC1.VIN; no longer C14.2, VOLTAGEREG.EN, VOLTAGEREG.IN
- net AGND: now also R11.1
- net DGND: now also C11.1, C12.1, IC1.GND; no longer C1.1, C2.1, R11.1, U1.GND@PAD, VOLTAGEREG.GND
- net N$6: now also C13.2; no longer C1.2
- net N$7: now also C12.2; no longer C2.2
- net RX: now also U1.PD0(RXD); no longer U1.PD1(TXD)
- net TX: now also U1.PD1(TXD); no longer U1.PD0(RXD)
Other:
- moved on the sheet: C14

Commit message: started board
started pcb layout
Parts:
- JST_MOTOR_1: value JST_CONNECTOR_FEMALE -> JST_MOTOR_1
- renumbered U$1 to JST_MOTOR_1
Changed lines of the file:
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@@
 <?xml version="1.0" encoding="utf-8"?>
 <!DOCTYPE eagle SYSTEM "eagle.dtd">
-<eagle version="8.0.1">
+<eagle version="8.4.1">
 <drawing>
 <settings>
 <setting alwaysvectorfont="no"/>
+<setting keepoldvectorfont="yes"/>
 <setting verticaltext="up"/>
 </settings>
@@
 <part name="R10" library="SparkFun-Resistors" deviceset="10.5KOHM1/10W1%(0603)" device="" value="10k"/>
 <part name="R11" library="SparkFun-Resistors" deviceset="10.5KOHM1/10W1%(0603)" device="" value="10k"/>
-<part name="U$1" library="JST_CONNECTOR_FEMALE. through hole" deviceset="JST_CONNECTOR_FEMALE" device=""/>
+<part name="JST_MOTOR_1" library="JST_CONNECTOR_FEMALE. through hole" deviceset="JST_CONNECTOR_FEMALE" device="" value="JST_MOTOR_1"/>
 <part name="U$3" library="JST_CONNECTOR_FEMALE. through hole" deviceset="JST_CONNECTOR_FEMALE" device=""/>
 <part name="U$4" library="JST_CONNECTOR_FEMALE. through hole" deviceset="JST_CONNECTOR_FEMALE" device=""/>
@@
 <instance part="R10" gate="G$1" x="271.78" y="88.9" rot="R90"/>
 <instance part="R11" gate="G$1" x="271.78" y="73.66" rot="R90"/>
-<instance part="U$1" gate="G$1" x="-17.78" y="96.52" rot="R270"/>
+<instance part="JST_MOTOR_1" gate="G$1" x="-17.78" y="96.52" rot="R270"/>
 <instance part="U$3" gate="G$1" x="-63.5" y="96.52" rot="R270"/>
 <instance part="U$4" gate="G$1" x="-66.04" y="40.64" rot="R270"/>
@@
 <junction x="-33.02" y="106.68"/>
 <label x="-33.02" y="111.76" size="1.778" layer="95" xref="yes"/>
-<pinref part="U$1" gate="G$1" pin="+"/>
+<pinref part="JST_MOTOR_1" gate="G$1" pin="+"/>
 <wire x1="-33.02" y1="99.06" x2="-27.94" y2="99.06" width="0.1524" layer="91"/>
 </segment>
@@
 <wire x1="-27.94" y1="91.44" x2="-45.72" y2="91.44" width="0.1524" layer="91"/>
 <junction x="-45.72" y="91.44"/>
-<pinref part="U$1" gate="G$1" pin="-"/>
+<pinref part="JST_MOTOR_1" gate="G$1" pin="-"/>
 <wire x1="-27.94" y1="91.44" x2="-27.94" y2="93.98" width="0.1524" layer="91"/>
 </segment>
